File: fab/KiCad/SqueakCheck.kicad_pcb (KiCad board)
At the start: 2 copper layers, 98 x 80 mm, 64 parts, among them J1 J1 command harness, J2 J2 power harness, J3 J3 audio harness, J4 RCJ-2123, SW1 94HBB16T hex dial, SW2 PLAY B3F-1000, SW3 RESET B3F-1000

Commit message: Rev E.6: hex dial fits with its 0 at the top
The Grayhill 94HBB16T fits SW1's holes either way round. E.5's pin map
assumed 0 toward the bottom, so a switch fitted with 0 at the top swapped
SOUND0<->SOUND1 and SOUND2<->SOUND3. E.6 turns the footprint's pin numbers
180 degrees and swaps the four sound tracks where they meet the resistors;
hole positions are unchanged.

- Gerbers: rerouted S0-S3 tracks (filleted), three small back-pour
  keep-outs, silk "0"/"8" at the dial, REV E.6
- KiCad PCB/schematic updated to match (tracks verified against Gerbers)
- Schematic PDF: rev and SW1 orientation note
- Board renders, website, README, fab notes and BOM updated
- Raster DRC: netlist matches, no islands, clearance unchanged from E.5

Co-Authored-By: Claude Opus 5.5 <noreply@anthropic.com>
Claude-Session: https://claude.ai/code/session_012k9RuKwdgXoTh4kCDBBGuh
Routing:
- net S3: track 20.1 -> 48.2 mm
- net S2: track 44.7 -> 23.6 mm
- net S1: track 24.4 -> 37.0 mm
- net S0: track 33.5 -> 24.4 mm
