File: fab/KiCad/SqueakCheck.kicad_sch (KiCad schematic)
At the start: 27 parts, among them J1 J1 command harness, J2 J2 power harness, J3 J3 audio harness, J4 RCJ-2123, SW1 94HBB16T hex dial, SW2 PLAY B3F-1000, SW3 RESET B3F-1000

Commit message: Rev E.6: hex dial fits with its 0 at the top
The Grayhill 94HBB16T fits SW1's holes either way round. E.5's pin map
assumed 0 toward the bottom, so a switch fitted with 0 at the top swapped
SOUND0<->SOUND1 and SOUND2<->SOUND3. E.6 turns the footprint's pin numbers
180 degrees and swaps the four sound tracks where they meet the resistors;
hole positions are unchanged.

- Gerbers: rerouted S0-S3 tracks (filleted), three small back-pour
  keep-outs, silk "0"/"8" at the dial, REV E.6
- KiCad PCB/schematic updated to match (tracks verified against Gerbers)
- Schematic PDF: rev and SW1 orientation note
- Board renders, website, README, fab notes and BOM updated
- Raster DRC: netlist matches, no islands, clearance unchanged from E.5

Co-Authored-By: Claude Opus 5.5 <noreply@anthropic.com>
Claude-Session: https://claude.ai/code/session_012k9RuKwdgXoTh4kCDBBGuh
Changed lines of the file:
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@@
 (kicad_sch (version 20231120) (generator "eeschema") (generator_version "8.0") (paper "A2")
-  (title_block (title "Squeak Check!") (rev "E.5") (company "Ethical Paul") (comment 1 "Generated from the board netlist; see Schematic_RevE5.pdf for the drawn schematic"))
+  (title_block (title "Squeak Check!") (rev "E.6") (company "Ethical Paul") (comment 1 "Generated from the board netlist; see Schematic_RevE6.pdf for the drawn schematic"))
   (symbol (lib_id "SqueakCheck:J1") (at 40.64 40.64 0) (unit 1) (exclude_from_sim no) (in_bom yes) (on_board yes) (dnp no)
     (property "Reference" "J1" (at 40.64 26.67 0) (effects (font (size 1.27 1.27))))
@@
   )
   (wire (pts (xy 149.86 173.99) (xy 144.78 173.99)) (stroke (width 0) (type default)))
-  (label "S1" (at 144.78 173.99 0) (fields_autoplaced yes) (effects (font (size 1.27 1.27)) (justify right bottom)))
+  (label "S0" (at 144.78 173.99 0) (fields_autoplaced yes) (effects (font (size 1.27 1.27)) (justify right bottom)))
   (wire (pts (xy 149.86 176.53) (xy 144.78 176.53)) (stroke (width 0) (type default)))
   (label "+5V" (at 144.78 176.53 0) (fields_autoplaced yes) (effects (font (size 1.27 1.27)) (justify right bottom)))
   (wire (pts (xy 149.86 179.07) (xy 144.78 179.07)) (stroke (width 0) (type default)))
-  (label "S3" (at 144.78 179.07 0) (fields_autoplaced yes) (effects (font (size 1.27 1.27)) (justify right bottom)))
+  (label "S2" (at 144.78 179.07 0) (fields_autoplaced yes) (effects (font (size 1.27 1.27)) (justify right bottom)))
   (wire (pts (xy 149.86 181.61) (xy 144.78 181.61)) (stroke (width 0) (type default)))
-  (label "S2" (at 144.78 181.61 0) (fields_autoplaced yes) (effects (font (size 1.27 1.27)) (justify right bottom)))
+  (label "S3" (at 144.78 181.61 0) (fields_autoplaced yes) (effects (font (size 1.27 1.27)) (justify right bottom)))
   (wire (pts (xy 149.86 184.15) (xy 144.78 184.15)) (stroke (width 0) (type default)))
   (label "+5V" (at 144.78 184.15 0) (fields_autoplaced yes) (effects (font (size 1.27 1.27)) (justify right bottom)))
   (wire (pts (xy 149.86 186.69) (xy 144.78 186.69)) (stroke (width 0) (type default)))
-  (label "S0" (at 144.78 186.69 0) (fields_autoplaced yes) (effects (font (size 1.27 1.27)) (justify right bottom)))
+  (label "S1" (at 144.78 186.69 0) (fields_autoplaced yes) (effects (font (size 1.27 1.27)) (justify right bottom)))
   (symbol (lib_id "SqueakCheck:PWR1") (at 220.98 180.34 0) (unit 1) (exclude_from_sim no) (in_bom yes) (on_board yes) (dnp no)
     (property "Reference" "PWR1" (at 220.98 172.72 0) (effects (font (size 1.27 1.27))))
